Commit message: Backup -> tutorial finished

File: src/mec_mobile/mec_mobile_description/urdf/robots/robot_3d.urdf.xacro (robot description, xacro)
@@ -1,4 +1,4 @@
 <?xml version="1.0"?>
-<robot name="my_robot" xmlns:xacro="http://www.ros.org/wiki/xacro" xmlns:gz="http://gazebosim.org/schema">
+<robot name="robot_3d" xmlns:xacro="http://www.ros.org/wiki/xacro" xmlns:gz="http://gazebosim.org/schema">
     <xacro:property name="M_PI" value="3.1415926535897931" />
     <xacro:arg name="robot_name" default="robot_3d"/>
@@ -55,5 +55,5 @@
       topic_name="imu/data"/>
     <!-- Gazebo frictions -->
-    <gazebo reference='front_left_wheel'>
+    <gazebo reference='front_left_wheel_link'>
       <collision>
         <surface>
@@ -68,5 +68,5 @@
       </collision>
     </gazebo>
-    <gazebo reference='back_left_wheel'>
+    <gazebo reference='back_left_wheel_link'>
       <collision>
         <surface>
@@ -81,5 +81,5 @@
       </collision>
     </gazebo>
-    <gazebo reference='front_right_wheel'>
+    <gazebo reference='front_right_wheel_link'>
       <collision>
         <surface>
@@ -94,5 +94,5 @@
       </collision>
     </gazebo>
-    <gazebo reference='back_right_wheel'>
+    <gazebo reference='back_right_wheel_link'>
       <collision>
         <surface>
@@ -110,4 +110,5 @@
       <mu1>0.000002</mu1>
       <mu2>0.000002</mu2>
+      <!-- <material>Gazebo/Red</material> -->
     </gazebo>
     <!--
